File: KLogShield/InterfaceEagle/interfaceBoard.brd (EAGLE design)
At the start: 50.8 x 61 mm, 10 parts, among them T1 2N2222, X1 1751280, X2 1751280, X3 1751303, X4 1751303, X5 1751303, X6 1751303, X7 1751248

Commit message: klog interface board gen2
Parts:
- added R2: 470, adafruit:M0805
- R1: value 4.7K -> 100; device adafruit:0207/9 -> adafruit:M0805
- moved X5 46.0 mm to (45.7, 38.1)
- moved X7 45.2 mm to (6.86, 6.35)
- moved X6 32.7 mm to (6.10, 35.6), turned to 270 degrees
- moved R1 24.5 mm to (8.89, 17.3), turned to 90 degrees
- moved T1 23.8 mm to (15.5, 15.7), turned to 270 degrees
- moved JP1 20.2 mm to (31.0, 38.9)
- moved X3 19.2 mm to (21.8, 55.9), turned to 180 degrees
- moved X4 19.1 mm to (15.2, 35.6), turned to 270 degrees
- moved X2 13.1 mm to (25.1, 13.5), turned to 270 degrees
- moved X1 6.53 mm to (35.6, 13.5), turned to 270 degrees
Connections:
- removed net MOI5V: T1.E, X1.1, X1.4, X2.1, X2.4
- removed net PWR: R1.2, T1.B, X7.1, X7.2
- new net MOIGND: T1.C, X1.2, X1.5, X2.2, X2.5
- new net N$7: R1.1, R2.2, T1.B
- net 5V: now also R2.1, X1.1, X1.4, X2.1, X2.4, X7.1, X7.2; no longer T1.C
- net GND: now also R1.2, T1.E; no longer R1.1, X1.2, X1.5, X2.2, X2.5
- net M11: now also X2.3; no longer X1.3
- net M12: now also X1.3; no longer X1.6
- net M13: now also X2.6; no longer X2.3
- net M14: now also X1.6; no longer X2.6
Routing:
- net 5V: track 134.1 -> 256.2 mm
- net GND: track 235.6 -> 162.6 mm
- net M11: track 81.3 -> 28.9 mm
- net MOI5V: track 52.3 -> 0.00 mm
- net MOIGND: track 0.00 -> 48.1 mm
- net PWR: track 22.8 -> 0.00 mm
- net N$3: track 21.7 -> 0.00 mm
- net ADC11: track 38.1 -> 16.8 mm
- net N$2: track 15.3 -> 0.00 mm
- net ADC12: track 37.0 -> 22.0 mm
- net ADC24: track 7.74 -> 22.6 mm, vias 2 -> 0
- net ADC14: track 26.3 -> 41.1 mm
- net ADC23: track 7.77 -> 21.6 mm, vias 2 -> 0
- net N$7: track 0.00 -> 11.6 mm
- net M14: track 26.7 -> 37.4 mm
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